Commit message: dr_drift: Regenerate dr_drift model
Fix command to generate the car model in documentation
generate_dr_drift is located under gazebo_simulation

File: simulation/src/gazebo_simulation/param/car_specs/dr_drift/model.urdf (robot description, URDF)
Before this commit: robot dr_drift, 6 links, 5 joints
Links:
- link chassis: mass 4.8 -> 2.855
Joints:
- joint front_camera_joint: origin xyz=-0.006256036655947976 0.0017242800000000001 0.2645206675581313 rpy=0.0 0.15771603452297908 0.0 -> xyz=-0.006642588303756858 -0.0051331 0.26190124401903253 rpy=0.0 0.15614472561323053 0.0
